Commit message: Add {prefix} to robot urdf file.

File: ur10cranfield/urdf/ur10cranfield_1.urdf.xacro (robot description, xacro)
@@ -39,4 +39,6 @@
   <xacro:arg name="EE_name" default="none"/>
   <xacro:property name="EE_name" value="$(arg EE_name)"/>
+  <xacro:arg name="prefix" default=""/>
+  <xacro:property name="prefix" value="$(arg prefix)"/>
   <!-- UR10 Control ARGUMENTS -->
   <xacro:arg name="script_filename" default="none"/>
@@ -56,4 +58,5 @@
     input_recipe_filename="${input_recipe_filename}"
     output_recipe_filename="${output_recipe_filename}"
+    prefix="${prefix}"
   />
   <!-- Load ROS 2 Gazebo Plugin -->
@@ -70,5 +73,5 @@
   <link name="world"/>
   <!-- Robot TABLE: LINK -->
-  <link name='ur10_table'>
+  <link name='${prefix}ur10_table'>
     <visual>
       <origin xyz="0.0 0.0 0.0" rpy="0 0 0" />
@@ -92,13 +95,13 @@
   </link>
   <!-- Robot TABLE: FIXED JOINT -->
-  <joint name="world_joint" type="fixed">
+  <joint name="${prefix}world_joint" type="fixed">
     <parent link="world" />
-    <child link = "ur10_table" />
+    <child link = "${prefix}ur10_table" />
     <origin xyz="0.0 0.0 0.0" rpy="0.0 0.0 0.0" />
   </joint>
   <!-- Robot TABLE: Robot+TABLE JOINT -->
-  <joint name="ur_joint" type="fixed">
-    <parent link="ur10_table" />
-    <child link = "base_link" />
+  <joint name="${prefix}ur_joint" type="fixed">
+    <parent link="${prefix}ur10_table" />
+    <child link = "${prefix}base_link" />
     <origin xyz="0.0 0.0 0.91" rpy="0.0 0.0 0.0" />
   </joint>

Commit message: Add (prefix) to urdf files.

File: ur10cranfield/urdf/ur10cranfield_1.urdf.xacro (robot description, xacro)
@@ -39,4 +39,6 @@
   <xacro:arg name="EE_name" default="none"/>
   <xacro:property name="EE_name" value="$(arg EE_name)"/>
+  <xacro:arg name="prefix" default=""/>
+  <xacro:property name="prefix" value="$(arg prefix)"/>
   <!-- UR10 Control ARGUMENTS -->
   <xacro:arg name="script_filename" default="none"/>
@@ -56,4 +58,5 @@
     input_recipe_filename="${input_recipe_filename}"
     output_recipe_filename="${output_recipe_filename}"
+    prefix="${prefix}"
   />
   <!-- Load ROS 2 Gazebo Plugin -->
@@ -69,5 +72,5 @@
   <link name="world"/>
   <!-- Robot TABLE: LINK -->
-  <link name='ur10_table'>
+  <link name='${prefix}ur10_table'>
     <visual>
       <origin xyz="0.0 0.0 0.0" rpy="0 0 0" />
@@ -91,13 +94,13 @@
   </link>
   <!-- Robot TABLE: FIXED JOINT -->
-  <joint name="world_joint" type="fixed">
+  <joint name="${prefix}world_joint" type="fixed">
     <parent link="world" />
-    <child link = "ur10_table" />
+    <child link = "${prefix}ur10_table" />
     <origin xyz="0.0 0.0 0.0" rpy="0.0 0.0 0.0" />
   </joint>
   <!-- Robot TABLE: Robot+TABLE JOINT -->
-  <joint name="ur_joint" type="fixed">
-    <parent link="ur10_table" />
-    <child link = "base_link" />
+  <joint name="${prefix}ur_joint" type="fixed">
+    <parent link="${prefix}ur10_table" />
+    <child link = "${prefix}base_link" />
     <origin xyz="0.0 0.0 0.91" rpy="0.0 0.0 0.0" />
   </joint>
